File: target-6-board.kicad_pcb (KiCad board)
At the start: 2 copper layers, 99.1 x 75.4 mm, 42 parts, among them J1 Conn_01x10_Socket, J10 RJ14, J11 RJ14, J12 RJ14, J13 RJ14, J14 RJ14, J15 RJ14, J2 Conn_01x12_Socket, J3 Conn_01x10_Socket, J4 Conn_01x12_Socket, J9 RJ14, Q0 NMOS, Q1 NMOS, Q2 NMOS, Q3 NMOS, Q4 NMOS, Q5 NMOS, Q6 NMOS, Q7 NMOS

Commit message: PCB order version
- Add USB connectors for power supply to M5Stamp C3
- Add RJ14 connectors for multiplay
Parts:
- added D6: D_TVS, Diode_SMD:D_SOD-323, F.Cu at (105.4, 95.5)
- added D7: D_TVS, Diode_SMD:D_SOD-323, F.Cu at (101.8, 101.6)
- added H1: MountingHole, MountingHole:MountingHole_3.2mm_M3_ISO14580, F.Cu at (30.5, 109.2)
- added H2: MountingHole, MountingHole:MountingHole_3.2mm_M3_ISO14580, F.Cu at (119.4, 109.2)
- added H3: MountingHole, MountingHole:MountingHole_3.2mm_M3_ISO14580, F.Cu at (30.5, 58.4)
- added H4: MountingHole, MountingHole:MountingHole_3.2mm_M3_ISO14580, F.Cu at (119.4, 47.0)
- added J12: RJ14, Connector_RJ:RJ14_Connfly_DS1133-S4_Horizontal, F.Cu at (114.3, 73.9)
- added J13: RJ14, Connector_RJ:RJ14_Connfly_DS1133-S4_Horizontal, F.Cu at (114.3, 90.4)
- added J14: USB_A, Connector_USB:USB_A_Molex_67643_Horizontal, F.Cu at (59.7, 102.9)
- added J15: USB_A, Connector_USB:USB_A_Molex_67643_Horizontal, F.Cu at (82.5, 102.9)
- added J16: USB_C_Receptacle_PowerOnly_6P, Connector_USB:USB_C_Receptacle_GCT_USB4125-xx-x_6P_TopMnt_Horizontal, F.Cu at (105.9, 113.5)
- added R18: 5.1K, Resistor_SMD:R_0603_1608Metric, F.Cu at (112.6, 104.1)
- added R19: 5.1K, Resistor_SMD:R_0603_1608Metric, F.Cu at (112.6, 101.6)
- moved D0 17.3 mm to (47.0, 89.3)
- moved R17 8.89 mm to (106.2, 54.6)
- moved D1 8.89 mm to (41.9, 57.5)
- moved J11 1.27 mm to (114.3, 57.4)
- renumbered J14 to J10, J15 to J11, J9 to J5, J10 to J6, J11 to J7, J12 to J8, J13 to J9
Connections:
- D0 pad 1: C_GPIO0 -> C_GPIO10
- J2 pad 10: C_GPIO5 -> CLOW_OUT
- J2 pad 11: C_GPIO4 -> CLOW_IN
- J2 pad 6: unconnected-(J2-Pin_6-Pad6) -> C_GPIO10
- J2 pad 8: unconnected-(J2-Pin_8-Pad8) -> CHIGH_OUT
- J2 pad 9: unconnected-(J2-Pin_9-Pad9) -> CHIGH_IN
- J4 pad 1: C_GPIO0 -> C_GPIO10
- J5 pad 3: C_GPIO0 -> C_GPIO10
- Q6 pad 3: C_GPIO4 -> C_GPIO0
- Q7 pad 3: C_GPIO5 -> C_GPIO1
- R14 pad 2: C_GPIO4 -> C_GPIO0
- R16 pad 2: C_GPIO5 -> C_GPIO1
Routing:
- net Net-(D6-A1): track 0.00 -> 104.5 mm
- net C_GPIO1: track 0.00 -> 95.8 mm, vias 0 -> 2
- net CHIGH_IN: track 0.00 -> 89.4 mm, vias 0 -> 3
- net C_GPIO5: track 80.7 -> 0.00 mm, vias 2 -> 0
- net CHIGH_OUT: track 0.00 -> 80.3 mm, vias 0 -> 2
- net C_GPIO10: track 0.00 -> 70.7 mm, vias 0 -> 1
- net C_GPIO4: track 70.6 -> 0.00 mm, vias 2 -> 0
- net CLOW_OUT: track 0.00 -> 69.6 mm, vias 0 -> 1
- net CLOW_IN: track 0.00 -> 69.3 mm, vias 0 -> 1
- net C_GPIO0: track 49.8 -> 95.8 mm, vias 0 -> 2
- net SWITCH_BUTTON: track 33.7 -> 48.4 mm
- net Net-(J16-CC1): track 0.00 -> 12.9 mm, vias 0 -> 2
- net Net-(J16-CC2): track 0.00 -> 10.7 mm, vias 0 -> 2
- net S0_GPIO1: track 35.4 -> 42.8 mm
- net SWITCH_BUZZER: track 27.9 -> 30.4 mm, vias 2 -> 1
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Other:
- board size 99.1 x 75.4 mm -> 99.1 x 90.7 mm
