File: target-6-board.kicad_sch (KiCad schematic)
At the start: 55 parts, among them J1 Conn_01x10_Socket, J10 RJ14, J11 RJ14, J12 RJ14, J13 RJ14, J14 USB_A, J15 USB_A, J16 USB_C_Receptacle_PowerOnly_6P, J2 Conn_01x12_Socket, J3 Conn_01x10_Socket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

Commit message: fix NMOS type to BSS138 and PCB design
Parts:
- Q0, Q1, Q2, Q3, Q4, Q5, Q6, Q7: value NMOS -> Transistor_FET:BSS138; symbol Simulation_SPICE:NMOS -> Transistor_FET:BSS138
Connections:
- net C_GPIO0: now also Q6.2 (S); no longer Q6.3 (S)
- net C_GPIO1: now also Q7.2 (S); no longer Q7.3 (S)
- net C_VCC3V3: now also Q6.1 (G), Q7.1 (G); no longer Q6.2 (G), Q7.2 (G)
- net S0_GPIO10: now also Q2.2 (S); no longer Q2.3 (S)
- net S0_GPIO18: now also Q3.2 (S); no longer Q3.3 (S)
- net S0_GPIO19: now also Q4.2 (S); no longer Q4.3 (S)
- net S0_GPIO21: now also Q5.2 (S); no longer Q5.3 (S)
- net S0_GPIO8: now also Q0.2 (S); no longer Q0.3 (S)
- net S0_GPIO9: now also Q1.2 (S); no longer Q1.3 (S)
- net S0_VCC3V3: now also Q0.1 (G), Q1.1 (G), Q2.1 (G), Q3.1 (G), Q4.1 (G), Q5.1 (G); no longer Q0.2 (G), Q1.2 (G), Q2.2 (G), Q3.2 (G), Q4.2 (G), Q5.2 (G)
- net SWITCH_BUTTON: now also Q6.3 (D); no longer Q6.1 (D)
- net SWITCH_BUZZER: now also Q7.3 (D); no longer Q7.1 (D)
- net TARGET_LED0: now also Q0.3 (D); no longer Q0.1 (D)
- net TARGET_LED1: now also Q1.3 (D); no longer Q1.1 (D)
- net TARGET_LED2: now also Q2.3 (D); no longer Q2.1 (D)
- net TARGET_LED3: now also Q3.3 (D); no longer Q3.1 (D)
- net TARGET_LED4: now also Q4.3 (D); no longer Q4.1 (D)
- net TARGET_LED5: now also Q5.3 (D); no longer Q5.1 (D)
Changed lines of the file:
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@@
     )
   )
-  (symbol (lib_id "Simulation_SPICE:NMOS") (at 185.42 88.9 270) (unit 1)
+  (symbol (lib_id "Transistor_FET:BSS138") (at 185.42 88.9 270) (unit 1)
     (in_bom yes) (on_board yes) (dnp no) (fields_autoplaced)
     (property "Reference" "Q1" (at 185.42 95.25 90)
       (effects (font (size 1.27 1.27)))
     )
-    (property "Value" "NMOS" (at 185.42 97.79 90)
-      (effects (font (size 1.27 1.27)))
-    )
-    (property "Footprint" "Package_TO_SOT_SMD:SOT-23" (at 187.96 93.98 0)
-      (effects (font (size 1.27 1.27)) hide)
-    )
-    (property "Datasheet" "https://ngspice.sourceforge.io/docs/ngspice-html-manual/manual.xhtml#cha_MOSFETs" (at 172.72 88.9 0)
-      (effects (font (size 1.27 1.27)) hide)
+    (property "Value" "Transistor_FET:BSS138" (at 185.42 97.79 90)
+      (effects (font (size 1.27 1.27)))
+    )
+    (property "Footprint" "Package_TO_SOT_SMD:SOT-23" (at 183.515 93.98 0)
+      (effects (font (size 1.27 1.27) italic) (justify left) hide)
+    )
+    (property "Datasheet" "https://www.onsemi.com/pub/Collateral/BSS138-D.PDF" (at 181.61 93.98 0)
+      (effects (font (size 1.27 1.27)) (justify left) hide)
     )
     (property "Sim.Device" "NMOS" (at 168.275 88.9 0)
@@
     )
   )
-  (symbol (lib_id "Simulation_SPICE:NMOS") (at 185.42 39.37 270) (unit 1)
+  (symbol (lib_id "Transistor_FET:BSS138") (at 185.42 39.37 270) (unit 1)
     (in_bom yes) (on_board yes) (dnp no) (fields_autoplaced)
     (property "Reference" "Q4" (at 185.42 45.72 90)
       (effects (font (size 1.27 1.27)))
     )
-    (property "Value" "NMOS" (at 185.42 48.26 90)
-      (effects (font (size 1.27 1.27)))
-    )
-    (property "Footprint" "Package_TO_SOT_SMD:SOT-23" (at 187.96 44.45 0)
-      (effects (font (size 1.27 1.27)) hide)
-    )
-    (property "Datasheet" "https://ngspice.sourceforge.io/docs/ngspice-html-manual/manual.xhtml#cha_MOSFETs" (at 172.72 39.37 0)
-      (effects (font (size 1.27 1.27)) hide)
+    (property "Value" "Transistor_FET:BSS138" (at 185.42 48.26 90)
+      (effects (font (size 1.27 1.27)))
+    )
+    (property "Footprint" "Package_TO_SOT_SMD:SOT-23" (at 183.515 44.45 0)
+      (effects (font (size 1.27 1.27) italic) (justify left) hide)
+    )
+    (property "Datasheet" "https://www.onsemi.com/pub/Collateral/BSS138-D.PDF" (at 181.61 44.45 0)
+      (effects (font (size 1.27 1.27)) (justify left) hide)
     )
     (property "Sim.Device" "NMOS" (at 168.275 39.37 0)
@@
     )
   )
-  (symbol (lib_id "Simulation_SPICE:NMOS") (at 250.19 22.86 270) (unit 1)
+  (symbol (lib_id "Transistor_FET:BSS138") (at 250.19 22.86 270) (unit 1)
     (in_bom yes) (on_board yes) (dnp no) (fields_autoplaced)
     (property "Reference" "Q7" (at 250.19 29.21 90)
       (effects (font (size 1.27 1.27)))
     )
-    (property "Value" "NMOS" (at 250.19 31.75 90)
-      (effects (font (size 1.27 1.27)))
-    )
-    (property "Footprint" "Package_TO_SOT_SMD:SOT-23" (at 252.73 27.94 0)
-      (effects (font (size 1.27 1.27)) hide)
-    )
-    (property "Datasheet" "https://ngspice.sourceforge.io/docs/ngspice-html-manual/manual.xhtml#cha_MOSFETs" (at 237.49 22.86 0)
-      (effects (font (size 1.27 1.27)) hide)
+    (property "Value" "Transistor_FET:BSS138" (at 250.19 31.75 90)
+      (effects (font (size 1.27 1.27)))
+    )
+    (property "Footprint" "Package_TO_SOT_SMD:SOT-23" (at 248.285 27.94 0)
+      (effects (font (size 1.27 1.27) italic) (justify left) hide)
+    )
+    (property "Datasheet" "https://www.onsemi.com/pub/Collateral/BSS138-D.PDF" (at 246.38 27.94 0)
+      (effects (font (size 1.27 1.27)) (justify left) hide)
     )
     (property "Sim.Device" "NMOS" (at 233.045 22.86 0)
@@
     )
   )
-  (symbol (lib_id "Simulation_SPICE:NMOS") (at 185.42 105.41 270) (unit 1)
+  (symbol (lib_id "Transistor_FET:BSS138") (at 185.42 105.41 270) (unit 1)
     (in_bom yes) (on_board yes) (dnp no)
     (property "Reference" "Q0" (at 185.42 111.76 90)
       (effects (font (size 1.27 1.27)))
     )
-    (property "Value" "NMOS" (at 185.42 114.3 90)
-      (effects (font (size 1.27 1.27)))
-    )
-    (property "Footprint" "Package_TO_SOT_SMD:SOT-23" (at 187.96 110.49 0)
-      (effects (font (size 1.27 1.27)) hide)
-    )
-    (property "Datasheet" "https://ngspice.sourceforge.io/docs/ngspice-html-manual/manual.xhtml#cha_MOSFETs" (at 172.72 105.41 0)
-      (effects (font (size 1.27 1.27)) hide)
+    (property "Value" "Transistor_FET:BSS138" (at 185.42 114.3 90)
+      (effects (font (size 1.27 1.27)))
+    )
+    (property "Footprint" "Package_TO_SOT_SMD:SOT-23" (at 183.515 110.49 0)
+      (effects (font (size 1.27 1.27) italic) (justify left) hide)
+    )
+    (property "Datasheet" "https://www.onsemi.com/pub/Collateral/BSS138-D.PDF" (at 181.61 110.49 0)
+      (effects (font (size 1.27 1.27)) (justify left) hide)
     )
     (property "Sim.Device" "NMOS" (at 168.275 105.41 0)
@@
     )
   )
-  (symbol (lib_id "Simulation_SPICE:NMOS") (at 250.19 39.37 270) (unit 1)
+  (symbol (lib_id "Transistor_FET:BSS138") (at 250.19 39.37 270) (unit 1)
     (in_bom yes) (on_board yes) (dnp no) (fields_autoplaced)
     (property "Reference" "Q6" (at 250.19 45.72 90)
       (effects (font (size 1.27 1.27)))
     )
-    (property "Value" "NMOS" (at 250.19 48.26 90)
-      (effects (font (size 1.27 1.27)))
-    )
-    (property "Footprint" "Package_TO_SOT_SMD:SOT-23" (at 252.73 44.45 0)
-      (effects (font (size 1.27 1.27)) hide)
-    )
-    (property "Datasheet" "https://ngspice.sourceforge.io/docs/ngspice-html-manual/manual.xhtml#cha_MOSFETs" (at 237.49 39.37 0)
-      (effects (font (size 1.27 1.27)) hide)
+    (property "Value" "Transistor_FET:BSS138" (at 250.19 48.26 90)
+      (effects (font (size 1.27 1.27)))
+    )
+    (property "Footprint" "Package_TO_SOT_SMD:SOT-23" (at 248.285 44.45 0)
+      (effects (font (size 1.27 1.27) italic) (justify left) hide)
+    )
+    (property "Datasheet" "https://www.onsemi.com/pub/Collateral/BSS138-D.PDF" (at 246.38 44.45 0)
+      (effects (font (size 1.27 1.27)) (justify left) hide)
     )
     (property "Sim.Device" "NMOS" (at 233.045 39.37 0)
@@
     )
   )
-  (symbol (lib_id "Simulation_SPICE:NMOS") (at 185.42 22.86 270) (unit 1)
+  (symbol (lib_id "Transistor_FET:BSS138") (at 185.42 22.86 270) (unit 1)
     (in_bom yes) (on_board yes) (dnp no) (fields_autoplaced)
     (property "Reference" "Q5" (at 185.42 29.21 90)
       (effects (font (size 1.27 1.27)))
     )
-    (property "Value" "NMOS" (at 185.42 31.75 90)
-      (effects (font (size 1.27 1.27)))
-    )
-    (property "Footprint" "Package_TO_SOT_SMD:SOT-23" (at 187.96 27.94 0)
-      (effects (font (size 1.27 1.27)) hide)
-    )
-    (property "Datasheet" "https://ngspice.sourceforge.io/docs/ngspice-html-manual/manual.xhtml#cha_MOSFETs" (at 172.72 22.86 0)
-      (effects (font (size 1.27 1.27)) hide)
+    (property "Value" "Transistor_FET:BSS138" (at 185.42 31.75 90)
+      (effects (font (size 1.27 1.27)))
+    )
+    (property "Footprint" "Package_TO_SOT_SMD:SOT-23" (at 183.515 27.94 0)
+      (effects (font (size 1.27 1.27) italic) (justify left) hide)
+    )
+    (property "Datasheet" "https://www.onsemi.com/pub/Collateral/BSS138-D.PDF" (at 181.61 27.94 0)
+      (effects (font (size 1.27 1.27)) (justify left) hide)
     )
     (property "Sim.Device" "NMOS" (at 168.275 22.86 0)
@@
     )
   )
-  (symbol (lib_id "Simulation_SPICE:NMOS") (at 185.42 55.88 270) (unit 1)
+  (symbol (lib_id "Transistor_FET:BSS138") (at 185.42 55.88 270) (unit 1)
     (in_bom yes) (on_board yes) (dnp no) (fields_autoplaced)
     (property "Reference" "Q3" (at 185.42 62.23 90)
       (effects (font (size 1.27 1.27)))
     )
-    (property "Value" "NMOS" (at 185.42 64.77 90)
-      (effects (font (size 1.27 1.27)))
-    )
-    (property "Footprint" "Package_TO_SOT_SMD:SOT-23" (at 187.96 60.96 0)
-      (effects (font (size 1.27 1.27)) hide)
-    )
-    (property "Datasheet" "https://ngspice.sourceforge.io/docs/ngspice-html-manual/manual.xhtml#cha_MOSFETs" (at 172.72 55.88 0)
-      (effects (font (size 1.27 1.27)) hide)
+    (property "Value" "Transistor_FET:BSS138" (at 185.42 64.77 90)
+      (effects (font (size 1.27 1.27)))
+    )
+    (property "Footprint" "Package_TO_SOT_SMD:SOT-23" (at 183.515 60.96 0)
+      (effects (font (size 1.27 1.27) italic) (justify left) hide)
+    )
+    (property "Datasheet" "https://www.onsemi.com/pub/Collateral/BSS138-D.PDF" (at 181.61 60.96 0)
+      (effects (font (size 1.27 1.27)) (justify left) hide)
     )
     (property "Sim.Device" "NMOS" (at 168.275 55.88 0)
@@
     )
   )
-  (symbol (lib_id "Simulation_SPICE:NMOS") (at 185.42 72.39 270) (unit 1)
+  (symbol (lib_id "Transistor_FET:BSS138") (at 185.42 72.39 270) (unit 1)
     (in_bom yes) (on_board yes) (dnp no) (fields_autoplaced)
     (property "Reference" "Q2" (at 185.42 78.74 90)
       (effects (font (size 1.27 1.27)))
     )
-    (property "Value" "NMOS" (at 185.42 81.28 90)
-      (effects (font (size 1.27 1.27)))
-    )
-    (property "Footprint" "Package_TO_SOT_SMD:SOT-23" (at 187.96 77.47 0)
-      (effects (font (size 1.27 1.27)) hide)
-    )
-    (property "Datasheet" "https://ngspice.sourceforge.io/docs/ngspice-html-manual/manual.xhtml#cha_MOSFETs" (at 172.72 72.39 0)
-      (effects (font (size 1.27 1.27)) hide)
+    (property "Value" "Transistor_FET:BSS138" (at 185.42 81.28 90)
+      (effects (font (size 1.27 1.27)))
+    )
+    (property "Footprint" "Package_TO_SOT_SMD:SOT-23" (at 183.515 77.47 0)
+      (effects (font (size 1.27 1.27) italic) (justify left) hide)
+    )
+    (property "Datasheet" "https://www.onsemi.com/pub/Collateral/BSS138-D.PDF" (at 181.61 77.47 0)
+      (effects (font (size 1.27 1.27)) (justify left) hide)
     )
     (property "Sim.Device" "NMOS" (at 168.275 72.39 0)
