File: ctrl/target-6-board-ctrl.kicad_pcb (KiCad board)
At the start: 2 copper layers, 37.9 x 46.8 mm, 17 parts, among them J1 RJ25, Q1 2SC1815, Q2 2SC1815, Q3 2SC1815

Commit message: ctrl: add mouting hole and board name and version
Parts:
- added H3: MountingHole, MountingHole:MountingHole_3.2mm_M3, F.Cu at (85.1, 30.5)
- added H4: MountingHole, MountingHole:MountingHole_3.2mm_M3, F.Cu at (85.1, 69.8)
- moved H1 39.7 mm to (43.2, 30.5)
- moved H2 35.6 mm to (43.2, 69.8)
Other:
- board size 37.9 x 46.8 mm -> 49.3 x 46.8 mm
- board text added: "target-6-ctrl v1.0-rc2"
Changed lines of the file:
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@@
   )
   (footprint "MountingHole:MountingHole_3.2mm_M3" (layer "F.Cu")
-    (at 48.26 69.85)
+    (at 43.18 30.48)
     (descr "Mounting Hole 3.2mm, no annular, M3")
     (tags "mounting hole 3.2mm no annular m3")
@@
         (effects (font (size 1 1) (thickness 0.15)))
     )
-    (fp_text value "MountingHole" (at 0 4.2) (layer "F.Fab")
+    (fp_text value "MountingHole" (at 0 -5.08) (layer "F.Fab")
         (effects (font (size 1 1) (thickness 0.15)))
     )
@@
   )
   (footprint "MountingHole:MountingHole_3.2mm_M3" (layer "F.Cu")
-    (at 78.74 69.85)
+    (at 43.18 69.85)
     (descr "Mounting Hole 3.2mm, no annular, M3")
     (tags "mounting hole 3.2mm no annular m3")
@@
     )
   )
+  (footprint "MountingHole:MountingHole_3.2mm_M3" (layer "F.Cu")
+    (at 85.09 30.48)
+    (descr "Mounting Hole 3.2mm, no annular, M3")
+    (tags "mounting hole 3.2mm no annular m3")
+    (property "Sheetfile" "target-6-board-ctrl.kicad_sch")
+    (property "Sheetname" "")
+    (property "ki_description" "Mounting Hole without connection")
+    (property "ki_keywords" "mounting hole")
+    (attr exclude_from_pos_files)
+    (fp_text reference "H3" (at 0 -4.2) (layer "F.SilkS") hide
+        (effects (font (size 1 1) (thickness 0.15)))
+    )
+    (fp_text value "MountingHole" (at 0 -5.08) (layer "F.Fab")
+        (effects (font (size 1 1) (thickness 0.15)))
+    )
+    (fp_text user "${REFERENCE}" (at 0 0) (layer "F.Fab")
+        (effects (font (size 1 1) (thickness 0.15)))
+    )
+    (fp_circle (center 0 0) (end 3.2 0)
+      (stroke (width 0.15) (type solid)) (fill none) (layer "Cmts.User"))
+    (fp_circle (center 0 0) (end 3.45 0)
+      (stroke (width 0.05) (type solid)) (fill none) (layer "F.CrtYd"))
+    (pad "" np_thru_hole circle (at 0 0) (size 3.2 3.2) (drill 3.2) (layers "*.Cu" "*.Mask"))
+  )
   (footprint "Resistor_THT:R_Axial_DIN0207_L6.3mm_D2.5mm_P7.62mm_Horizontal" (layer "F.Cu")
     (at 60.96 45.72 -90)
@@
       (rotate (xyz 0 0 0))
     )
+  )
+  (footprint "MountingHole:MountingHole_3.2mm_M3" (layer "F.Cu")
+    (at 85.09 69.85)
+    (descr "Mounting Hole 3.2mm, no annular, M3")
+    (tags "mounting hole 3.2mm no annular m3")
+    (property "Sheetfile" "target-6-board-ctrl.kicad_sch")
+    (property "Sheetname" "")
+    (property "ki_description" "Mounting Hole without connection")
+    (property "ki_keywords" "mounting hole")
+    (attr exclude_from_pos_files)
+    (fp_text reference "H4" (at 0 -4.2) (layer "F.SilkS") hide
+        (effects (font (size 1 1) (thickness 0.15)))
+    )
+    (fp_text value "MountingHole" (at 0 4.2) (layer "F.Fab")
+        (effects (font (size 1 1) (thickness 0.15)))
+    )
+    (fp_text user "${REFERENCE}" (at 0 0) (layer "F.Fab")
+        (effects (font (size 1 1) (thickness 0.15)))
+    )
+    (fp_circle (center 0 0) (end 3.2 0)
+      (stroke (width 0.15) (type solid)) (fill none) (layer "Cmts.User"))
+    (fp_circle (center 0 0) (end 3.45 0)
+      (stroke (width 0.05) (type solid)) (fill none) (layer "F.CrtYd"))
+    (pad "" np_thru_hole circle (at 0 0) (size 3.2 3.2) (drill 3.2) (layers "*.Cu" "*.Mask"))
   )
   (footprint "Resistor_THT:R_Axial_DIN0207_L6.3mm_D2.5mm_P7.62mm_Horizontal" (layer "F.Cu")
@@
     )
   )
-  (gr_rect (start 44.45 26.67) (end 82.353354 73.463354)
+  (gr_rect (start 39.37 26.67) (end 88.703354 73.463354)
     (stroke (width 0.05) (type default)) (fill none) (layer "Edge.Cuts"))
+  (gr_text "target-6-ctrl\nv1.0-rc2" (at 43.18 34.29 90) (layer "F.SilkS")
+    (effects (font (size 1 1) (thickness 0.1)) (justify right bottom))
+  )
   (segment (start 69.85 66.04) (end 63.5 66.04) (width 0.2) (layer "F.Cu") (net 1))
   (segment (start 55.88 53.34) (end 55.88 58.36) (width 0.2) (layer "F.Cu") (net 1))
@@
     (polygon
       (pts
-        (xy 44.45 26.67)
-        (xy 44.45 73.66)
-        (xy 85.09 73.66)
-        (xy 85.09 26.67)
+        (xy 39.37 26.67)
+        (xy 39.37 73.66)
+        (xy 90.17 73.66)
+        (xy 90.17 26.67)
       )
     )
@@
     (polygon
       (pts
-        (xy 44.45 26.67)
-        (xy 44.45 73.66)
-        (xy 85.09 73.66)
-        (xy 85.09 26.67)
+        (xy 39.37 26.67)
+        (xy 39.37 73.66)
+        (xy 90.17 73.66)
+        (xy 90.17 26.67)
       )
     )
